File: Design/LM35/LM35_Remote.sch (EAGLE design)
At the start: 0 parts

Commit message: Trabajo realizado el dia miercoles 3 septiembre
Parts:
- added 2N2907: (no value), transistor:2N2907A-PNP-TO18-EBC
- added D1: 1N4148DO35-7, diode:1N4148DO35-7
- added JP1: (no value), pinhead:PINHD-1X2
- added LM317: (no value), v-reg:LM317TS
- added LM35: LM50, linear:LM50
- added R1: 402, resistor:R-EU_0207_7
- added R2: 50, resistor:R-TRIMM3296W
- added R3: 62.5, resistor:R-EU_0207_7
- added R4: 4.7K, resistor:R-EU_0207_7
Connections:
- new net N$1: 2N2907.B, LM35.+VS, R4.1
- new net N$2: 2N2907.C, LM35.VO, R3.2
- new net N$3: 2N2907.E, D1.C, LM317.IN, R4.2
- new net N$4: JP1.2, LM317.ADJ, R2.A, R3.1
- new net N$5: R1.1, R2.E
- new net N$6: LM317.OUT, R1.2
- new net N$7: LM35.GND, R2.S
- new net N$8: D1.A, JP1.1
Changed lines of the file:
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@@
 <grid distance="0.1" unitdist="inch" unit="inch" style="lines" multiple="1" display="no" altdistance="0.01" altunitdist="inch" altunit="inch"/>
 <layers>
+<layer number="1" name="Top" color="4" fill="1" visible="yes" active="no"/>
+<layer number="16" name="Bottom" color="1" fill="1" visible="yes" active="no"/>
+<layer number="17" name="Pads" color="2" fill="1" visible="yes" active="no"/>
+<layer number="18" name="Vias" color="2" fill="1" visible="yes" active="no"/>
+<layer number="19" name="Unrouted" color="6" fill="1" visible="yes" active="no"/>
+<layer number="20" name="Dimension" color="15" fill="1" visible="yes" active="no"/>
+<layer number="21" name="tPlace" color="7" fill="1" visible="yes" active="no"/>
+<layer number="22" name="bPlace" color="7" fill="1" visible="yes" active="no"/>
+<layer number="23" name="tOrigins" color="15" fill="1" visible="yes" active="no"/>
+<layer number="24" name="bOrigins" color="15" fill="1" visible="yes" active="no"/>
+<layer number="25" name="tNames" color="7" fill="1" visible="yes" active="no"/>
+<layer number="26" name="bNames" color="7" fill="1" visible="yes" active="no"/>
+<layer number="27" name="tValues" color="7" fill="1" visible="yes" active="no"/>
+<layer number="28" name="bValues" color="7" fill="1" visible="yes" active="no"/>
+<layer number="29" name="tStop" color="7" fill="3" visible="no" active="no"/>
+<layer number="30" name="bStop" color="7" fill="6" visible="no" active="no"/>
+<layer number="31" name="tCream" color="7" fill="4" visible="no" active="no"/>
+<layer number="32" name="bCream" color="7" fill="5" visible="no" active="no"/>
+<layer number="33" name="tFinish" color="6" fill="3" visible="no" active="no"/>
+<layer number="34" name="bFinish" color="6" fill="6" visible="no" active="no"/>
+<layer number="35" name="tGlue" color="7" fill="4" visible="no" active="no"/>
+<layer number="36" name="bGlue" color="7" fill="5" visible="no" active="no"/>
+<layer number="37" name="tTest" color="7" fill="1" visible="yes" active="no"/>
+<layer number="38" name="bTest" color="7" fill="1" visible="yes" active="no"/>
+<layer number="39" name="tKeepout" color="4" fill="11" visible="no" active="no"/>
+<layer number="40" name="bKeepout" color="1" fill="11" visible="no" active="no"/>
+<layer number="41" name="tRestrict" color="4" fill="10" visible="no" active="no"/>
+<layer number="42" name="bRestrict" color="1" fill="10" visible="no" active="no"/>
+<layer number="43" name="vRestrict" color="2" fill="10" visible="no" active="no"/>
+<layer number="44" name="Drills" color="7" fill="1" visible="no" active="no"/>
+<layer number="45" name="Holes" color="7" fill="1" visible="no" active="no"/>
+<layer number="46" name="Milling" color="3" fill="1" visible="yes" active="no"/>
+<layer number="47" name="Measures" color="7" fill="1" visible="yes" active="no"/>
+<layer number="48" name="Document" color="7" fill="1" visible="yes" active="no"/>
+<layer number="49" name="Reference" color="7" fill="1" visible="yes" active="no"/>
+<layer number="51" name="tDocu" color="7" fill="1" visible="yes" active="no"/>
+<layer number="52" name="bDocu" color="7" fill="1" visible="yes" active="no"/>
 <layer number="90" name="Modules" color="5" fill="1" visible="yes" active="yes"/>
 <layer number="91" name="Nets" color="2" fill="1" visible="yes" active="yes"/>
@@
 <layer number="97" name="Info" color="7" fill="1" visible="yes" active="yes"/>
 <layer number="98" name="Guide" color="6" fill="1" visible="yes" active="yes"/>
+<layer number="99" name="SpiceOrder" color="5" fill="1" visible="yes" active="yes"/>
 </layers>
 <schematic xreflabel="%F%N/%S.%C%R" xrefpart="/%S.%C%R">
@@
 </classes>
 <parts>
+<part name="LM317" library="v-reg" deviceset="LM317TS" device=""/>
+<part name="R1" library="resistor" deviceset="R-EU_" device="0207_7" value="402"/>
+<part name="R2" library="resistor" deviceset="R-TRIMM" device="3296W" value="50"/>
+<part name="2N2907" library="transistor" deviceset="*-PNP-" device="TO18-EBC" technology="2N2907A"/>
+<part name="LM35" library="linear" deviceset="LM50" device=""/>
+<part name="R3" library="resistor" deviceset="R-EU_" device="0207_7" value="62.5"/>
+<part name="R4" library="resistor" deviceset="R-EU_" device="0207_7" value="4.7K"/>
+<part name="D1" library="diode" deviceset="1N4148" device="DO35-7"/>
+<part name="JP1" library="pinhead" deviceset="PINHD-1X2" device=""/>
 </parts>
 <sheets>
@@
 </plain>
 <instances>
+<instance part="LM317" gate="1" x="40.64" y="109.22" rot="MR0"/>
+<instance part="R1" gate="G$1" x="33.02" y="99.06" rot="R90"/>
+<instance part="R2" gate="G$1" x="33.02" y="71.12" rot="R180"/>
+<instance part="2N2907" gate="G$1" x="-2.54" y="101.6" rot="MR0"/>
+<instance part="LM35" gate="G$1" x="12.7" y="88.9" rot="MR270"/>
+<instance part="R3" gate="G$1" x="-5.08" y="68.58" rot="R90"/>
+<instance part="R4" gate="G$1" x="12.7" y="109.22" rot="R90"/>
+<instance part="D1" gate="G$1" x="60.96" y="116.84" rot="R180"/>
+<instance part="JP1" gate="G$1" x="78.74" y="91.44"/>
 </instances>
 <busses>
 </busses>
 <nets>
+<net name="N$1" class="0">
+<segment>
+<pinref part="R4" gate="G$1" pin="1"/>
+<pinref part="LM35" gate="G$1" pin="+VS"/>
+<wire x1="12.7" y1="104.14" x2="12.7" y2="101.6" width="0.1524" layer="91"/>
+<pinref part="2N2907" gate="G$1" pin="B"/>
+<wire x1="12.7" y1="101.6" x2="12.7" y2="99.06" width="0.1524" layer="91"/>
+<wire x1="0" y1="101.6" x2="12.7" y2="101.6" width="0.1524" layer="91"/>
+</segment>
+</net>
+<net name="N$2" class="0">
+<segment>
+<pinref part="2N2907" gate="G$1" pin="C"/>
+<wire x1="-5.08" y1="96.52" x2="-5.08" y2="78.74" width="0.1524" layer="91"/>
+<pinref part="LM35" gate="G$1" pin="VO"/>
+<wire x1="-5.08" y1="78.74" x2="12.7" y2="78.74" width="0.1524" layer="91"/>
+<pinref part="R3" gate="G$1" pin="2"/>
+<wire x1="-5.08" y1="73.66" x2="-5.08" y2="78.74" width="0.1524" layer="91"/>
+</segment>
+</net>
+<net name="N$3" class="0">
+<segment>
+<pinref part="R4" gate="G$1" pin="2"/>
+<wire x1="48.26" y1="116.84" x2="12.7" y2="116.84" width="0.1524" layer="91"/>
+<wire x1="12.7" y1="116.84" x2="12.7" y2="114.3" width="0.1524" layer="91"/>
+<wire x1="12.7" y1="116.84" x2="-5.08" y2="116.84" width="0.1524" layer="91"/>
+<wire x1="-5.08" y1="116.84" x2="-5.08" y2="106.68" width="0.1524" layer="91"/>
+<pinref part="LM317" gate="1" pin="IN"/>
+<wire x1="48.26" y1="109.22" x2="48.26" y2="116.84" width="0.1524" layer="91"/>
+<pinref part="D1" gate="G$1" pin="C"/>
+<wire x1="48.26" y1="116.84" x2="58.42" y2="116.84" width="0.1524" layer="91"/>
+<pinref part="2N2907" gate="G$1" pin="E"/>
+</segment>
+</net>
+<net name="N$4" class="0">
+<segment>
+<pinref part="R3" gate="G$1" pin="1"/>
+<wire x1="-5.08" y1="63.5" x2="-5.08" y2="58.42" width="0.1524" layer="91"/>
+<pinref part="R2" gate="G$1" pin="A"/>
+<wire x1="-5.08" y1="58.42" x2="33.02" y2="58.42" width="0.1524" layer="91"/>
+<wire x1="33.02" y1="58.42" x2="33.02" y2="66.04" width="0.1524" layer="91"/>
+<pinref part="LM317" gate="1" pin="ADJ"/>
+<wire x1="40.64" y1="101.6" x2="40.64" y2="58.42" width="0.1524" layer="91"/>
+<wire x1="40.64" y1="58.42" x2="33.02" y2="58.42" width="0.1524" layer="91"/>
+<wire x1="40.64" y1="58.42" x2="76.2" y2="58.42" width="0.1524" layer="91"/>
+<pinref part="JP1" gate="G$1" pin="2"/>
+<wire x1="76.2" y1="58.42" x2="76.2" y2="91.44" width="0.1524" layer="91"/>
+</segment>
+</net>
+<net name="N$5" class="0">
+<segment>
+<pinref part="R2" gate="G$1" pin="E"/>
+<wire x1="33.02" y1="76.2" x2="33.02" y2="93.98" width="0.1524" layer="91"/>
+<pinref part="R1" gate="G$1" pin="1"/>
+</segment>
+</net>
+<net name="N$6" class="0">
+<segment>
+<pinref part="LM317" gate="1" pin="OUT"/>
+<pinref part="R1" gate="G$1" pin="2"/>
+<wire x1="33.02" y1="109.22" x2="33.02" y2="104.14" width="0.1524" layer="91"/>
+</segment>
+</net>
+<net name="N$7" class="0">
+<segment>
+<pinref part="LM35" gate="G$1" pin="GND"/>
+<pinref part="R2" gate="G$1" pin="S"/>
+<wire x1="20.32" y1="88.9" x2="27.94" y2="88.9" width="0.1524" layer="91"/>
+<wire x1="27.94" y1="88.9" x2="27.94" y2="71.12" width="0.1524" layer="91"/>
+</segment>
+</net>
+<net name="N$8" class="0">
+<segment>
+<pinref part="D1" gate="G$1" pin="A"/>
+<pinref part="JP1" gate="G$1" pin="1"/>
+<wire x1="63.5" y1="116.84" x2="76.2" y2="116.84" width="0.1524" layer="91"/>
+<wire x1="76.2" y1="116.84" x2="76.2" y2="93.98" width="0.1524" layer="91"/>
+</segment>
+</net>
 </nets>
 </sheet>
